Commit message: EDIT: code name and README.md

File: src/mecanum_pkg/mecanum_robot_description/urdf/mecanum_robot_velodyne_height_2m/mecanum_frame.urdf.xacro (robot description, xacro)
@@ -58,5 +58,5 @@
   <!--******************* add VLP laser Link *************************************-->
     <joint name="VLP16_base_mount_joint" type="fixed">
-      <origin xyz="0 0.0 2" rpy="0.0 0.0 0.0"/>
+      <origin xyz="0 0.0 0.5" rpy="0.0 0.0 0.0"/>
       <parent link="base_link"/>
       <child link="VLP16_base_link"/>
